File: 3S_LiPo.kicad_sch (KiCad schematic)
At the start: 0 parts

Commit message: REV1 PCB that was sent to production (PCBWAY)
Parts:
- added BT1, BT2, BT3: Battery_Cell, symbol Device:Battery_Cell
Connections:
- new net: BT1.2 (-), BT2.1 (+)
- new net: BT2.2 (-), BT3.1 (+)
