File: untitled.kicad_sch (KiCad schematic)
At the start: 32 parts, among them Q6 NMOS, Q7 NMOS, Q8 NMOS, Q9 NMOS

Commit message: REV1 PCB that was sent to production (PCBWAY)
Parts:
- removed C30: C, symbol Device:C
- removed Q8: NMOS, symbol Simulation_SPICE:NMOS
- removed R47, R48, R49, R50: R_US, symbol Device:R_US
- C26, C27, C28, C29: value C -> 0.1u
- R39, R40: value R_US -> 5.1k
Connections:
- net 3P: now also C26.1, D13.2 (A), Q6.3 (S), R34.1
- net PACK+: now reaches C27.2, C28.2, D14.2 (A), D15.2 (A), E3.2, Q7.3 (S), Q9.3 (S), R35.1, R41.1, R43.1, R44.1
- net at Q7.2 (G), R35.2, R37.1: now also D14.1 (K)
- net at Q7.1 (D): now also Q6.1 (D)
