File: MAIN.kicad_pcb (KiCad board)
At the start: 2 copper layers, 125 x 85 mm, 207 parts, among them J1 USB_C_Receptacle_USB2.0_16P, J2 Conn_01x07_Socket, J3 Conn_01x07_Socket, J4 Conn_01x02_Socket, J5 Conn_01x07_Socket, J6 Conn_01x04_Socket, Q1 DMG2302UK-7, Q10 PSMN1R0-30YLDX, Q11 PSMN1R0-30YLDX, Q12 PSMN1R0-30YLDX, Q13 PSMN1R0-30YLDX, Q14 PSMN1R0-30YLDX, Q15 PSMN1R0-30YLDX, Q2 DMG2302UK-7, Q3 DMG2302UK-7, Q4 BSS123, Q5 ZXMP10A13FTA, Q6 FDD4141, Q7 FDD4141, Q8 PSMN1R0-30YLDX, SW1 SW_Push, SW2 SW_Push, SW3 SPDT_Slide_PTH_11.6x4.0mm, U1 ESP32-S3-WROOM-1, U2 TPS62170DSG, U3 BQ76952PFBR, U4 TLV62569DBV

Commit message: These files are for the final report
NOTE:
1. PCB has mixed up nets so many traces going to the BQ76952 are DISCONNECTED.
2. BOTH active and passive balancing are connected in parallel even though only active balancing is supposed to be connected.
Routing:
- net 3P: track 212.9 -> 207.8 mm
Changed lines of the file:
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@@
-	(segment
-		(start 78.0252 96.907)
-		(end 78.0252 101.3478)
-		(width 0.2)
-		(layer "F.Cu")
-		(net "3P")
-	)
 	(segment
 		(start 78.0252 96.907)
@@
 		(width 0.2)
 		(layer "F.Cu")
-		(net "3P")
-	)
-	(segment
-		(start 78.0252 101.3478)
-		(end 77.509 101.864)
-		(width 0.2)
-		(layer "F.Cu")
